File: hardware/cardiac.sch (KiCad schematic (older format))
At the start: 15 parts, among them IC1 ATTINY45-P, SW1 NF, U1 LM7805, U2 LM386

Commit message: Revised
Parts:
- added R1: 220R, symbol R
Connections:
- net GND: now also R1.2; no longer D1.2 (K), D2.2 (K)
- new net: D1.2 (K), D2.2 (K), R1.1
- no-connect marks 0 -> 4
Changed lines of the file:
@@
-EESchema Schematic File Version 2  date Tue 19 Jan 2016 12:19:41 AM BRST
+EESchema Schematic File Version 2  date Tue 19 Jan 2016 10:47:40 AM BRST
 LIBS:power
 LIBS:device
@@
 Comment4 ""
 $EndDescr
+$Comp
+L GND #PWR?
+U 1 1 569E3044
+P 5800 5500
+F 0 "#PWR?" H 5800 5500 30  0001 C CNN
+F 1 "GND" H 5800 5430 30  0001 C CNN
+	1    5800 5500
+	0    -1   -1   0
+$EndComp
+Wire Wire Line
+	5200 5500 5300 5500
+Wire Wire Line
+	6700 3900 6700 3650
+Wire Wire Line
+	6700 3650 6200 3650
+Wire Wire Line
+	6200 3650 6200 3100
+Wire Wire Line
+	8200 5150 8200 4500
+Connection ~ 5900 5000
+Connection ~ 6200 3100
+Wire Wire Line
+	5900 5000 5900 5150
+Wire Wire Line
+	4800 5500 4800 5200
+Wire Wire Line
+	8150 3350 8150 3100
+Wire Wire Line
+	8150 3100 7900 3100
+Connection ~ 4750 3100
+Wire Wire Line
+	5000 3100 2850 3100
+Wire Wire Line
+	2850 3100 2850 4100
+Wire Wire Line
+	6050 3100 6050 3650
+Wire Wire Line
+	4750 3100 4750 3650
+Wire Wire Line
+	4800 5200 4700 5200
+Wire Wire Line
+	6900 4700 6900 5200
+Wire Wire Line
+	6900 5200 6800 5200
+Wire Wire Line
+	7300 4800 7300 4300
+Wire Wire Line
+	7300 4300 7550 4300
+Wire Wire Line
+	7950 4300 8200 4300
+Connection ~ 8200 4800
+Wire Wire Line
+	6800 4700 6800 4800
+Connection ~ 5200 5500
+Wire Wire Line
+	7200 3100 7300 3100
+Wire Wire Line
+	5650 3650 5150 3650
+Connection ~ 5400 3650
+Wire Wire Line
+	6200 3100 5800 3100
+Connection ~ 6050 3100
+Wire Wire Line
+	5400 3800 5400 3400
+Wire Wire Line
+	5550 4200 6300 4200
+Wire Wire Line
+	5550 4600 5550 4900
+Wire Wire Line
+	5550 4900 4700 4900
+Wire Wire Line
+	4700 4900 4700 5200
+Wire Wire Line
+	5900 4200 5900 4600
 Connection ~ 5900 4200
 Wire Wire Line
-	5900 4200 5900 4600
-Wire Wire Line
-	4700 4900 4700 5200
-Wire Wire Line
-	4700 4900 5550 4900
-Wire Wire Line
-	5550 4900 5550 4600
-Wire Wire Line
-	5550 4200 6300 4200
-Wire Wire Line
-	6200 3900 6200 3100
-Wire Wire Line
-	6200 3900 6700 3900
-Wire Wire Line
-	5400 3800 5400 3400
-Connection ~ 6050 3100
-Wire Wire Line
-	6200 3100 5800 3100
-Connection ~ 5400 3650
-Wire Wire Line
-	5650 3650 5150 3650
-Wire Wire Line
-	7200 3100 7300 3100
-Connection ~ 6300 4700
-Wire Wire Line
-	6700 4700 6300 4700
-Connection ~ 5200 5500
-Wire Wire Line
-	5200 5750 5200 5200
-Wire Wire Line
-	6800 4700 6800 4800
-Connection ~ 8200 4800
-Wire Wire Line
-	7950 4300 8200 4300
-Wire Wire Line
-	7550 4300 7300 4300
-Wire Wire Line
-	7300 4300 7300 4800
-Wire Wire Line
-	6800 5200 6900 5200
-Wire Wire Line
-	6900 5200 6900 4700
-Wire Wire Line
-	4700 5200 4800 5200
-Wire Wire Line
-	6300 4400 6300 5150
-Wire Wire Line
-	4750 3100 4750 3650
-Wire Wire Line
-	6050 3100 6050 3650
-Wire Wire Line
-	2850 4100 2850 3100
-Wire Wire Line
-	2850 3100 5000 3100
-Connection ~ 4750 3100
-Wire Wire Line
-	2850 4600 2850 5100
-Wire Wire Line
-	8200 5150 8200 4500
-Wire Wire Line
-	7900 3100 8150 3100
-Wire Wire Line
-	8150 3100 8150 3350
-Wire Wire Line
-	4800 5200 4800 5500
-Wire Wire Line
-	5900 5000 5900 5150
-$Comp
-L GND #PWR?
+	5200 5200 5300 5200
+Wire Wire Line
+	5300 5200 5300 5500
+$Comp
+L R R1
+U 1 1 569E2FDD
+P 5550 5500
+F 0 "R1" V 5630 5500 50  0000 C CNN
+F 1 "220R" V 5550 5500 50  0000 C CNN
+	1    5550 5500
+	0    -1   -1   0
+$EndComp
+$Comp
+L GND #PWR01
+U 1 1 569E27C5
+P 2850 4600
+F 0 "#PWR01" H 2850 4600 30  0001 C CNN
+F 1 "GND" H 2850 4530 30  0001 C CNN
+	1    2850 4600
+	0    1    1    0
+$EndComp
+$Comp
+L GND #PWR02
+U 1 1 569E2768
+P 6300 4400
+F 0 "#PWR02" H 6300 4400 30  0001 C CNN
+F 1 "GND" H 6300 4330 30  0001 C CNN
+	1    6300 4400
+	0    1    -1   0
+$EndComp
+$Comp
+L GND #PWR03
+U 1 1 569E275A
+P 6700 4700
+F 0 "#PWR03" H 6700 4700 30  0001 C CNN
+F 1 "GND" H 6700 4630 30  0001 C CNN
+	1    6700 4700
+	1    0    0    -1
+$EndComp
+NoConn ~ 5550 4500
+NoConn ~ 5550 4400
+NoConn ~ 5550 4300
+NoConn ~ 5550 4100
+$Comp
+L GND #PWR04
 U 1 1 569D9BD8
 P 5900 5150
-F 0 "#PWR?" H 5900 5150 30  0001 C CNN
+F 0 "#PWR04" H 5900 5150 30  0001 C CNN
 F 1 "GND" H 5900 5080 30  0001 C CNN
 	1    5900 5150
@@
 $EndComp
 $Comp
-L GND #PWR01
+L GND #PWR05
 U 1 1 569CE647
 P 8150 3350
-F 0 "#PWR01" H 8150 3350 30  0001 C CNN
+F 0 "#PWR05" H 8150 3350 30  0001 C CNN
 F 1 "GND" H 8150 3280 30  0001 C CNN
 	1    8150 3350
@@
 $EndComp
 $Comp
-L GND #PWR02
+L GND #PWR06
 U 1 1 569CE5E1
 P 8200 5150
-F 0 "#PWR02" H 8200 5150 30  0001 C CNN
+F 0 "#PWR06" H 8200 5150 30  0001 C CNN
 F 1 "GND" H 8200 5080 30  0001 C CNN
 	1    8200 5150
@@
 $EndComp
 $Comp
-L GND #PWR03
-U 1 1 569CE5D5
-P 2850 5100
-F 0 "#PWR03" H 2850 5100 30  0001 C CNN
-F 1 "GND" H 2850 5030 30  0001 C CNN
-	1    2850 5100
-	1    0    0    -1
-$EndComp
-$Comp
-L GND #PWR04
+L GND #PWR07
 U 1 1 569CE5B2
 P 5400 3800
-F 0 "#PWR04" H 5400 3800 30  0001 C CNN
+F 0 "#PWR07" H 5400 3800 30  0001 C CNN
 F 1 "GND" H 5400 3730 30  0001 C CNN
 	1    5400 3800
@@
 $EndComp
 $Comp
-L GND #PWR05
-U 1 1 569CE450
-P 6300 5150
-F 0 "#PWR05" H 6300 5150 30  0001 C CNN
-F 1 "GND" H 6300 5080 30  0001 C CNN
-	1    6300 5150
-	1    0    0    -1
-$EndComp
-$Comp
-L GND #PWR06
-U 1 1 569CE41E
-P 5200 5750
-F 0 "#PWR06" H 5200 5750 30  0001 C CNN
-F 1 "GND" H 5200 5680 30  0001 C CNN
-	1    5200 5750
-	1    0    0    -1
-$EndComp
-$Comp

Commit message: The old schemas were wrong
Parts:
- added R3: 10K, symbol R
Connections:
- net labels added: +5V, +9V
- wire segments 31 -> 29
- no-connect marks 4 -> 3
Other:
- moved on the sheet: BT1, C1, C2, SW1, U1
Changed lines of the file:
@@
-EESchema Schematic File Version 2  date Tue 19 Jan 2016 10:47:40 AM BRST
+EESchema Schematic File Version 2  date Sun 24 Jan 2016 10:44:02 PM BRST
 LIBS:power
 LIBS:device
@@
 Sheet 1 1
 Title "Cardiac"
-Date "19 jan 2016"
+Date "25 jan 2016"
 Rev ""
 Comp "Pinewoods"
@@
 $EndDescr
 $Comp
-L GND #PWR?
+L +9V #PWR01
+U 1 1 56A56F1F
+P 6700 3900
+F 0 "#PWR01" H 6700 3870 20  0001 C CNN
+F 1 "+9V" H 6700 4010 30  0000 C CNN
+	1    6700 3900
+	1    0    0    -1
+$EndComp
+$Comp
+L GND #PWR02
+U 1 1 56A56EF9
+P 6100 4100
+F 0 "#PWR02" H 6100 4100 30  0001 C CNN
+F 1 "GND" H 6100 4030 30  0001 C CNN
+	1    6100 4100
+	0    -1   -1   0
+$EndComp
+$Comp
+L +5V #PWR03
+U 1 1 56A56EE0
+P 2850 4600
+F 0 "#PWR03" H 2850 4690 20  0001 C CNN
+F 1 "+5V" H 2850 4690 30  0000 C CNN
+	1    2850 4600
+	0    -1   -1   0
+$EndComp
+$Comp
+L GND #PWR04
+U 1 1 56A56ECE
+P 2850 4100
+F 0 "#PWR04" H 2850 4100 30  0001 C CNN
+F 1 "GND" H 2850 4030 30  0001 C CNN
+	1    2850 4100
+	0    1    1    0
+$EndComp
+$Comp
+L +9V #PWR05
+U 1 1 56A56E9B
+P 5300 2550
+F 0 "#PWR05" H 5300 2520 20  0001 C CNN
+F 1 "+9V" H 5300 2660 30  0000 C CNN
+	1    5300 2550
+	-1   0    0    1
+$EndComp
+Wire Wire Line
+	5300 2550 5300 2300
+Wire Wire Line
+	5550 4100 5600 4100
+Wire Wire Line
+	5300 5200 5300 5500
+Wire Wire Line
+	5300 5200 5200 5200
+Connection ~ 5900 4200
+Wire Wire Line
+	5900 4600 5900 4200
+Wire Wire Line
+	4700 4900 4700 5200
+Wire Wire Line
+	4700 4900 5550 4900
+Wire Wire Line
+	5550 4900 5550 4600
+Wire Wire Line
+	6300 4200 5550 4200
+Wire Wire Line
+	4500 2600 4500 3000
+Connection ~ 5150 2300
+Wire Wire Line
+	5300 2300 4900 2300
+Connection ~ 4500 2850
+Wire Wire Line
+	4250 2850 4750 2850
+Wire Wire Line
+	6300 2300 6400 2300
+Connection ~ 5200 5500
+Wire Wire Line
+	6800 4700 6800 4800
+Connection ~ 8200 4800
+Wire Wire Line
+	7950 4300 8200 4300
+Wire Wire Line
+	7550 4300 7300 4300
+Wire Wire Line
+	7300 4300 7300 4800
+Wire Wire Line
+	6800 5200 6900 5200
+Wire Wire Line
+	6900 5200 6900 4700
+Wire Wire Line
+	4700 5200 4800 5200
+Wire Wire Line
+	3850 2850 3850 2300
+Wire Wire Line
+	5150 2300 5150 2850
+Connection ~ 3850 2300
+Wire Wire Line
+	7000 2300 7250 2300
+Wire Wire Line
+	7250 2300 7250 2550
+Wire Wire Line
+	4800 5200 4800 5500
+Wire Wire Line
+	5900 5000 5900 5150
+Connection ~ 5900 5000
+Wire Wire Line
+	8200 4500 8200 5150
+Wire Wire Line
+	5300 5500 5200 5500
+Wire Wire Line
+	4100 2300 3750 2300
+$Comp
+L +5V #PWR06
+U 1 1 56A56E54
+P 3750 2300
+F 0 "#PWR06" H 3750 2390 20  0001 C CNN
+F 1 "+5V" H 3750 2390 30  0000 C CNN
+	1    3750 2300
+	0    -1   -1   0
+$EndComp
+$Comp
+L R R3
+U 1 1 56A56D4E
+P 5850 4100
+F 0 "R3" V 5930 4100 50  0000 C CNN
+F 1 "10K" V 5850 4100 50  0000 C CNN
+	1    5850 4100
+	0    -1   -1   0
+$EndComp
+$Comp
+L GND #PWR07
 U 1 1 569E3044
 P 5800 5500
-F 0 "#PWR?" H 5800 5500 30  0001 C CNN
+F 0 "#PWR07" H 5800 5500 30  0001 C CNN
 F 1 "GND" H 5800 5430 30  0001 C CNN
 	1    5800 5500
 	0    -1   -1   0
 $EndComp
-Wire Wire Line
-	5200 5500 5300 5500
-Wire Wire Line
-	6700 3900 6700 3650
-Wire Wire Line
-	6700 3650 6200 3650
-Wire Wire Line
-	6200 3650 6200 3100
-Wire Wire Line
-	8200 5150 8200 4500
-Connection ~ 5900 5000
-Connection ~ 6200 3100
-Wire Wire Line
-	5900 5000 5900 5150
-Wire Wire Line
-	4800 5500 4800 5200
-Wire Wire Line
-	8150 3350 8150 3100
-Wire Wire Line
-	8150 3100 7900 3100
-Connection ~ 4750 3100
-Wire Wire Line
-	5000 3100 2850 3100
-Wire Wire Line
-	2850 3100 2850 4100
-Wire Wire Line
-	6050 3100 6050 3650
-Wire Wire Line
-	4750 3100 4750 3650
-Wire Wire Line
-	4800 5200 4700 5200
-Wire Wire Line
-	6900 4700 6900 5200
-Wire Wire Line
-	6900 5200 6800 5200
-Wire Wire Line
-	7300 4800 7300 4300
-Wire Wire Line
-	7300 4300 7550 4300
-Wire Wire Line
-	7950 4300 8200 4300
-Connection ~ 8200 4800
-Wire Wire Line
-	6800 4700 6800 4800
-Connection ~ 5200 5500
-Wire Wire Line
-	7200 3100 7300 3100
-Wire Wire Line
-	5650 3650 5150 3650
-Connection ~ 5400 3650
-Wire Wire Line
-	6200 3100 5800 3100
-Connection ~ 6050 3100
-Wire Wire Line
-	5400 3800 5400 3400
-Wire Wire Line
-	5550 4200 6300 4200
-Wire Wire Line
-	5550 4600 5550 4900
-Wire Wire Line
-	5550 4900 4700 4900
-Wire Wire Line
-	4700 4900 4700 5200
-Wire Wire Line
-	5900 4200 5900 4600
-Connection ~ 5900 4200
-Wire Wire Line
-	5200 5200 5300 5200
-Wire Wire Line
-	5300 5200 5300 5500
 $Comp
 L R R1
@@
 $EndComp
 $Comp
-L GND #PWR01
-U 1 1 569E27C5
-P 2850 4600
-F 0 "#PWR01" H 2850 4600 30  0001 C CNN
-F 1 "GND" H 2850 4530 30  0001 C CNN
-	1    2850 4600
-	0    1    1    0
-$EndComp
-$Comp
-L GND #PWR02
+L GND #PWR08
 U 1 1 569E2768
 P 6300 4400
-F 0 "#PWR02" H 6300 4400 30  0001 C CNN
+F 0 "#PWR08" H 6300 4400 30  0001 C CNN
 F 1 "GND" H 6300 4330 30  0001 C CNN
 	1    6300 4400
@@
 $EndComp
 $Comp
-L GND #PWR03
+L GND #PWR09
 U 1 1 569E275A
 P 6700 4700
-F 0 "#PWR03" H 6700 4700 30  0001 C CNN
+F 0 "#PWR09" H 6700 4700 30  0001 C CNN
 F 1 "GND" H 6700 4630 30  0001 C CNN
 	1    6700 4700
@@
 NoConn ~ 5550 4400
 NoConn ~ 5550 4300
-NoConn ~ 5550 4100
-$Comp
-L GND #PWR04
+$Comp
+L GND #PWR010
 U 1 1 569D9BD8
 P 5900 5150
-F 0 "#PWR04" H 5900 5150 30  0001 C CNN
+F 0 "#PWR010" H 5900 5150 30  0001 C CNN
 F 1 "GND" H 5900 5080 30  0001 C CNN
 	1    5900 5150
@@
 $EndComp
 $Comp
-L GND #PWR05
+L GND #PWR011
 U 1 1 569CE647
-P 8150 3350
-F 0 "#PWR05" H 8150 3350 30  0001 C CNN
-F 1 "GND" H 8150 3280 30  0001 C CNN
-	1    8150 3350
-	1    0    0    -1
-$EndComp
-$Comp
-L GND #PWR06
+P 7250 2550
+F 0 "#PWR011" H 7250 2550 30  0001 C CNN
+F 1 "GND" H 7250 2480 30  0001 C CNN
+	1    7250 2550
+	1    0    0    -1
+$EndComp
+$Comp
+L GND #PWR012
 U 1 1 569CE5E1
 P 8200 5150
-F 0 "#PWR06" H 8200 5150 30  0001 C CNN
+F 0 "#PWR012" H 8200 5150 30  0001 C CNN
 F 1 "GND" H 8200 5080 30  0001 C CNN
 	1    8200 5150
@@
 $EndComp
 $Comp
-L GND #PWR07
+L GND #PWR013
 U 1 1 569CE5B2
-P 5400 3800
-F 0 "#PWR07" H 5400 3800 30  0001 C CNN
-F 1 "GND" H 5400 3730 30  0001 C CNN
-	1    5400 3800
+P 4500 3000
+F 0 "#PWR013" H 4500 3000 30  0001 C CNN
+F 1 "GND" H 4500 2930 30  0001 C CNN
+	1    4500 3000
 	1    0    0    -1
 $EndComp
@@
 L CP1 C2
 U 1 1 569CE50C
-P 4950 3650
-F 0 "C2" H 5000 3750 50  0000 L CNN
-F 1 "10uF" H 5000 3550 50  0000 L CNN
-F 2 "CP4" H 5000 3650 50  0000 C CNN
-	1    4950 3650
+P 4050 2850
+F 0 "C2" H 4100 2950 50  0000 L CNN
+F 1 "10uF" H 4100 2750 50  0000 L CNN
+F 2 "CP4" H 4100 2850 50  0000 C CNN
+	1    4050 2850
 	0    -1   -1   0
 $EndComp
@@
 L CP1 C1
 U 1 1 569CE506
-P 5850 3650
-F 0 "C1" H 5900 3750 50  0000 L CNN
-F 1 "220uF" H 5900 3550 50  0000 L CNN
-F 2 "CP36V" H 5900 3650 50  0000 C CNN
-	1    5850 3650
+P 4950 2850
+F 0 "C1" H 5000 2950 50  0000 L CNN
+F 1 "220uF" H 5000 2750 50  0000 L CNN
+F 2 "CP36V" H 5000 2850 50  0000 C CNN
+	1    4950 2850
 	0    1    1    0
 $EndComp
@@
 L BATTERY BT1
 U 1 1 569CDDCE
-P 7600 3100
-F 0 "BT1" H 7600 3300 50  0000 C CNN
-F 1 "BATTERY" H 7600 2910 50  0000 C CNN
-F 2 "bornier2" H 7600 3010 50  0000 C CNN
-	1    7600 3100
+P 6700 2300
+F 0 "BT1" H 6700 2500 50  0000 C CNN
+F 1 "BATTERY" H 6700 2110 50  0000 C CNN
+F 2 "bornier2" H 6700 2210 50  0000 C CNN
+	1    6700 2300
 	1    0    0    -1
 $EndComp
@@
 L SPST SW1
 U 1 1 569CDD9F
-P 6700 3100
-F 0 "SW1" H 6700 3200 70  0000 C CNN
-F 1 "NF" H 6700 3000 70  0000 C CNN
-F 2 "bornier2" H 6700 3100 70  0000 C CNN
-	1    6700 3100
+P 5800 2300
+F 0 "SW1" H 5800 2400 70  0000 C CNN
+F 1 "NF" H 5800 2200 70  0000 C CNN
+F 2 "bornier2" H 5800 2300 70  0000 C CNN
+	1    5800 2300
 	1    0    0    -1
 $EndComp
@@
 L LM7805 U1
 U 1 1 569CDAE8
-P 5400 3150
-F 0 "U1" H 5550 2954 60  0000 C CNN
-F 1 "LM7805" H 5400 3350 60  0000 C CNN
-F 2 "LM78XX" H 5400 3450 60  0000 C CNN
-	1    5400 3150
+P 4500 2350
+F 0 "U1" H 4650 2154 60  0000 C CNN
+F 1 "LM7805" H 4500 2550 60  0000 C CNN
+F 2 "LM78XX" H 4500 2650 60  0000 C CNN
+	1    4500 2350
 	-1   0    0    -1
 $EndComp
